File: LiPower.kicad_sch (KiCad schematic)
At the start: 28 parts, among them J4 TYPE-C-31-M-12, J5 Conn_01x02, Q1 AO3400A, U3 MAX77757, U7 PI3USB102EZLEX, U8 XC6206P332MR-G

Commit message: wired
Parts:
- renumbered C19 to C1, C23 to C14, C22 to C15, C20 to C18, C1 to C19, C18 to C2, C14 to C22, C2 to C23, C15 to C29, C21 to C30, D37 to D38, J4 to J1, Q1 to Q2, R24 to R12, R22 to R13, R23 to R14, R21 to R15, R20 to R16, R19 to R17, R25 to R18, U7 to U4, U3 to U5, U8 to U6
