File: Matrix.kicad_sch (KiCad schematic)
At the start: 69 parts, among them SW1 SW_Push, SW10 SW_Push, SW11 SW_Push, SW12 SW_Push, SW13 SW_Push, SW14 SW_Push, SW15 SW_Push, SW16 SW_Push, SW17 SW_Push, SW18 SW_Push, SW19 SW_Push, SW2 SW_Push, SW20 SW_Push, SW21 SW_Push, SW22 SW_Push, SW23 SW_Push, SW24 SW_Push, SW25 SW_Push, SW26 SW_Push, SW27 SW_Push, SW28 SW_Push, SW29 SW_Push, SW3 SW_Push, SW30 SW_Push, SW31 SW_Push, SW32 SW_Push, SW33 SW_Push, SW34 SW_Push, SW4 SW_Push, SW5 SW_Push, SW6 SW_Push, SW7 SW_Push, SW8 SW_Push, SW9 SW_Push

Commit message: wired
Parts:
- added C15: 100nF, Capacitor_SMD:C_0402_1005Metric, symbol Device:C
- added D38: D, Diode_SMD:D_SOD-323, symbol Device:D_Small
- added J9: Conn_01x02, Connector_PinHeader_2.54mm:PinHeader_1x02_P2.54mm_Vertical, symbol Connector_Generic:Conn_01x02
- added R24: 100k, Resistor_SMD:R_0402_1005Metric, symbol Device:R
Connections:
- net at D30.2 (A), SW30.2: now also D38.1 (K), J9.2 (Pin_2)
- new net +3V3: R24.1
- new net GND: C15.2, J9.1 (Pin_1)
- new net WAKEUP: C15.1, D38.2 (A), R24.2
Other:
- note added: "Pull COL0 down before going to sleep. Make the rest of them hi-Z."
