File: c47r.kicad_pcb (KiCad board)
At the start: 4 copper layers, 98 x 187 mm, 121 parts, among them J2 Conn_02x06_Top_Bottom, J3 OLED, J4 TYPE-C-31-M-12, J6 Conn_01x05, J7 SHF-105-01-L-D-RA, Q1 AO3400A, SW1 SW_Push, SW10 SW_Push, SW11 SW_Push, SW12 SW_Push, SW13 SW_Push, SW14 SW_Push, SW15 SW_Push, SW16 SW_Push, SW17 SW_Push, SW18 SW_Push, SW19 SW_Push, SW2 SW_Push, SW20 SW_Push, SW21 SW_Push, SW22 SW_Push, SW23 SW_Push, SW24 SW_Push, SW25 SW_Push, SW26 SW_Push, SW27 SW_Push, SW28 SW_Push, SW29 SW_Push, SW3 SW_Push, SW30 SW_Push, SW31 SW_Push, SW32 SW_Push, SW33 SW_Push, SW34 SW_Push, SW35 SW_Push, SW36 SW_Push, SW4 SW_Push, SW5 SW_Push, SW6 SW_Push, SW7 SW_Push, SW8 SW_Push, SW9 SW_Push, U1 RP2350A, U2 W25Q128JVSIQ, U8 XC6206P332MR-G, Y1 ABM8-272-T3

Commit message: hist
Parts:
- added C31: 4.7uF, Capacitor_SMD:C_0603_1608Metric, F.Cu at (159.4, 79.7)
- added J8: Conn_01x02, Connector_JST:JST_PH_S2B-PH-K_1x02_P2.00mm_Horizontal, F.Cu at (152.4, 80.8)

Commit message: wired
Parts:
- added C14: 4.7uF, Capacitor_SMD:C_0402_1005Metric, F.Cu at (106.0, 63.3)
- added C15: 100nF, Capacitor_SMD:C_0402_1005Metric, F.Cu at (74.3, 61.5)
- added C33: 4.7uF, Capacitor_SMD:C_0402_1005Metric, F.Cu at (64.5, 59.3)
- added D36: SS14, Diode_SMD:D_SMA, F.Cu at (90.0, 56.4)
- added D37: SS14, Diode_SMD:D_SMA, F.Cu at (79.2, 56.4)
- added D38: D, Diode_SMD:D_SOD-323, F.Cu at (74.8, 63.2)
- added D39: KT-0603W, LED_SMD:LED_0603_1608Metric, F.Cu at (62.0, 56.0)
- added J1: Conn_01x14, Connector_PinHeader_2.54mm:PinHeader_1x14_P2.54mm_Vertical, F.Cu at (109.8, 96.0)
- added J9: Conn_01x02, Connector_PinHeader_2.54mm:PinHeader_1x02_P2.54mm_Vertical, F.Cu at (68.0, 59.6)
- added R11: 5k1, Resistor_SMD:R_0402_1005Metric, F.Cu at (118.0, 57.6)
- added R19: 2k, Resistor_SMD:R_0402_1005Metric, F.Cu at (62.0, 57.5)
- added R20: 2k, Resistor_SMD:R_0402_1005Metric, F.Cu at (61.9, 59.3)
- added R24: 100k, Resistor_SMD:R_0402_1005Metric, F.Cu at (99.8, 73.9)
- added R3: 5k1, Resistor_SMD:R_0402_1005Metric, F.Cu at (113.2, 57.6)
- added U3: MCP73832-2-OT, Package_TO_SOT_SMD:SOT-23-5, F.Cu at (63.0, 62.2)
- C10, C31, C6, C7, C9: footprint Capacitor_SMD:C_0603_1608Metric -> Capacitor_SMD:C_0402_1005Metric
- R22, R23: value 1M -> 100k
- R5, R7, R8: footprint Resistor_SMD:R_0603_1608Metric -> Resistor_SMD:R_0402_1005Metric
- moved C31 97.5 mm to (63.0, 65.2), turned to 180 degrees
- moved SW36 93.1 mm to (153.3, 70.7), turned to -90 degrees
- moved SW35 91.6 mm to (153.4, 92.0)
- moved J8 91.6 mm to (61.5, 70.0)
- moved R4 88.2 mm to (150.0, 75.0), turned to -90 degrees
- moved D35 61.9 mm to (86.4, 56.4), turned to 90 degrees
- moved R22 39.7 mm to (67.1, 57.2), turned to 0 degrees
- moved R23 37.4 mm to (72.0, 58.3), turned to -90 degrees
- moved Q1 36.9 mm to (74.8, 58.8), turned to 180 degrees
- moved BZ1 30.3 mm to (93.3, 80.6), turned to -90 degrees
- moved C5 9.36 mm to (114.7, 70.0)
- moved R1 9.36 mm to (109.6, 68.0)
- moved R10 9.36 mm to (103.0, 71.7)
- moved R6 9.36 mm to (103.0, 73.9)
- moved R9 9.36 mm to (101.2, 73.9)
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Connections:
- BZ1 pad 1: /GPIO0 -> Net-(BZ1-+)
- C20 pad 1: /SYS -> +5V
- C31 pad 1: /BATT -> /Power/BATT
- C6 pad 1: +5V -> +3V3
- J4 pad A5: /CC1 -> /Power/CC1
- J4 pad B5: /CC2 -> /Power/CC2
- J8 pad 2: /BATT -> /Power/BATT
- Q1 pad 1: /EN_BUS_SENSE -> /Power/EN_BUS_SENSE
- R22 pad 1: /SYS -> /Power/BATT
- R9 pad 1: /GPIO0 -> WAKEUP
- U1 pad 2: /USB_SEL -> WAKEUP
- U1 pad 3: /GPIO0 -> Net-(BZ1-+)
- U1 pad 32: unconnected-(U1-GPIO20-Pad32) -> /Power/EN_BUS_SENSE
- U1 pad 33: unconnected-(U1-GPIO21-Pad33) -> /4N
- U1 pad 34: /4N -> /4P
- U1 pad 35: /4P -> /3N
- U1 pad 36: /3N -> /3P
- U1 pad 37: /3P -> /2N
- U1 pad 40: /2N -> /2P
- U1 pad 41: /2P -> /1N
- U1 pad 42: /1N -> /1P
- U1 pad 43: /1P -> /BUS_SENSE
- U1 pad 44: unconnected-(U1-ADC_AVDD-Pad44) -> +3V3
- U1 pad 49: +5V -> +3V3
- U1 pad 5: /D~{C} -> /SCK
- U1 pad 53: unconnected-(U1-USB_OTP_VDD-Pad53) -> +3V3
- U1 pad 7: /~{RES} -> /SDA
- U1 pad 8: /SDA -> /~{RES}
- U1 pad 9: /SCK -> /D~{C}
- U8 pad 3: /SYS -> +5V
Routing:
- net Net-(D30-A): track 9.08 -> 183.8 mm
- net Net-(D35-A): track 0.00 -> 91.1 mm
- net /BUS_SENSE: track 0.00 -> 69.9 mm, vias 0 -> 2
- net /Power/EN_BUS_SENSE: track 0.00 -> 69.5 mm, vias 0 -> 2
- net VBUS: track 0.00 -> 67.8 mm
- net COL4: track 119.7 -> 180.3 mm, vias 1 -> 0
- net /~{USB_BOOT}: track 0.00 -> 60.1 mm, vias 0 -> 2
- net GND: track 5.19 -> 63.7 mm, vias 8 -> 60
- net WAKEUP: track 0.00 -> 56.8 mm
- net /Power/BATT: track 0.00 -> 47.8 mm, vias 0 -> 1
- net /SWD: track 14.9 -> 53.1 mm
- net +3V3: track 9.41 -> 42.2 mm, vias 0 -> 15
- net +5V: track 0.00 -> 32.7 mm
- net /SWCLK: track 16.9 -> 49.2 mm
- net Net-(BZ1-+): track 0.00 -> 31.4 mm
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- added copper zone on In2.Cu, net +1V1
- added copper zone on F.Cu, net +3V3
- added copper zone on In1.Cu, net GND
- removed copper zone on F.Cu, net /VREG_LX
Other:
- outline, holes or cut-outs redrawn
- board text added: "GND"
