File: c47r.kicad_sch (KiCad schematic)
At the start: 54 parts, among them J2 Conn_02x06_Top_Bottom, J3 OLED, J4 TYPE-C-31-M-12, J6 Conn_01x05, J7 SHF-105-01-L-D-RA, J8 Conn_01x02, Q1 AO3400A, SW35 SW_Push, SW36 SW_Push, U1 RP2350A, U2 W25Q128JVSIQ, U8 XC6206P332MR-G, Y1 ABM8-272-T3

Commit message: wired
Parts:
- removed C20, C21: 100nF, Capacitor_SMD:C_0402_1005Metric, symbol Device:C
- removed C31: 4.7uF, Capacitor_SMD:C_0603_1608Metric, symbol Device:C
- removed J4: TYPE-C-31-M-12, Connector_USB:USB_C_Receptacle_HRO_TYPE-C-31-M-12, symbol Connector:USB_C_Receptacle_USB2.0_16P
- removed J8: Conn_01x02, Connector_JST:JST_PH_S2B-PH-K_1x02_P2.00mm_Horizontal, symbol Connector_Generic:Conn_01x02
- removed Q1: AO3400A, Package_TO_SOT_SMD:SOT-23, symbol Transistor_FET:AO3400A
- removed R22, R23: 1M, Resistor_SMD:R_0402_1005Metric, symbol Device:R
- removed U8: XC6206P332MR-G, Package_TO_SOT_SMD:SOT-23-3, symbol Regulator_Linear:XC6206PxxxMR
- added J1: Conn_01x14, Connector_PinHeader_2.54mm:PinHeader_1x14_P2.54mm_Vertical, symbol Connector_Generic:Conn_01x14
- C10, C6, C7, C9: footprint Capacitor_SMD:C_0603_1608Metric -> Capacitor_SMD:C_0402_1005Metric; LCSC (none) -> C23733
- C11, C12, C13, C24, C25, C26, C27, C28, C5, C8: LCSC (none) -> C1525; PN (none) -> CL05B104KO5NNNC
- D35: LCSC (none) -> C2480
- R5, R7, R8: footprint Resistor_SMD:R_0603_1608Metric -> Resistor_SMD:R_0402_1005Metric; LCSC C23140 -> (none)
Connections:
- net +3V3: now also C6.1, U1.44 (ADC_AVDD), U1.49 (VREG_VIN), U1.53 (USB_OTP_VDD), J1.14 (Pin_14)
- net +5V: no longer C6.1, U1.49 (VREG_VIN)
- net 1N: now also U1.41 (GPIO27/ADC1); no longer U1.42 (GPIO28/ADC2)
- net 1P: now also U1.42 (GPIO28/ADC2); no longer U1.43 (GPIO29/ADC3)
- net 2N: now also U1.37 (GPIO25); no longer U1.40 (GPIO26/ADC0)
- net 2P: now also U1.40 (GPIO26/ADC0); no longer U1.41 (GPIO27/ADC1)
- net 3N: now also U1.35 (GPIO23); no longer U1.36 (GPIO24)
- net 3P: now also U1.36 (GPIO24); no longer U1.37 (GPIO25)
- net 4N: now also U1.33 (GPIO21); no longer U1.34 (GPIO22)
- net 4P: now also U1.34 (GPIO22); no longer U1.35 (GPIO23)
- net BUS_SENSE: now also U1.43 (GPIO29/ADC3)
- net COL0: now also J1.2 (Pin_2)
- net COL1: now also J1.12 (Pin_12)
- net COL2: now also J1.11 (Pin_11)
- net COL3: now also J1.10 (Pin_10)
- net COL4: now also J1.5 (Pin_5)
- net D~{C}: now also U1.9 (GPIO6); no longer U1.5 (GPIO3)
- net GND: now also J1.13 (Pin_13)
- net ROW0: now also J1.9 (Pin_9)
- net ROW1: now also J1.8 (Pin_8)
- net ROW2: now also J1.7 (Pin_7)
- net ROW3: now also J1.6 (Pin_6)
- net ROW4: now also J1.4 (Pin_4)
- net ROW5: now also J1.3 (Pin_3)
- net ROW6: now also J1.1 (Pin_1)
- net SCK: now also U1.5 (GPIO3); no longer U1.9 (GPIO6)
- net SDA: now also U1.7 (GPIO4); no longer U1.8 (GPIO5)
- net ~{RES}: now also U1.8 (GPIO5); no longer U1.7 (GPIO4)
- net Power/EN_BUS_SENSE: now reaches U1.32 (GPIO20)
- net GPIO0: no longer names the net of BZ1.1 (+), U1.3 (GPIO1)
- net GPIO0: no longer R9.1
- net USB_SEL renamed WAKEUP
- net WAKEUP: now also R9.1
- no-connect marks 5 -> 3
Other:
- added sheet Power (Power.kicad_sch)
- note added: "Backup"
- note removed: "SPI6+PMOD8+ROW7+COL5+3POW"
- moved on the sheet: BZ1, C10, C12, C13, C24, C25, C26, C27, C28, C3, C4, C5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

Commit message: changes
Parts:
- BZ1, J7: now not fitted
Changed lines of the file:
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@@
 		(in_bom no)
 		(on_board yes)
-		(in_pos_files yes)
+		(in_pos_files no)
 		(dnp no)
 		(fields_autoplaced yes)
@@
 		(in_bom no)
 		(on_board yes)
-		(in_pos_files yes)
+		(in_pos_files no)
 		(dnp no)
 		(fields_autoplaced yes)
@@
 		(in_bom no)
 		(on_board yes)
-		(in_pos_files yes)
+		(in_pos_files no)
 		(dnp no)
 		(fields_autoplaced yes)
@@
 		(in_bom yes)
 		(on_board yes)
-		(in_pos_files yes)
-		(dnp no)
+		(in_pos_files no)
+		(dnp yes)
 		(fields_autoplaced yes)
 		(property "Reference" "BZ1"
@@
 		(in_bom no)
 		(on_board yes)
-		(in_pos_files yes)
+		(in_pos_files no)
 		(dnp no)
 		(fields_autoplaced yes)
@@
 		(in_bom no)
 		(on_board yes)
-		(in_pos_files yes)
+		(in_pos_files no)
 		(dnp no)
 		(fields_autoplaced yes)
@@
 		(in_bom no)
 		(on_board yes)
-		(in_pos_files yes)
+		(in_pos_files no)
 		(dnp no)
 		(fields_autoplaced yes)
@@
 		(in_bom no)
 		(on_board yes)
-		(in_pos_files yes)
+		(in_pos_files no)
 		(dnp no)
 		(fields_autoplaced yes)
@@
 		(in_bom yes)
 		(on_board yes)
-		(in_pos_files yes)
-		(dnp no)
+		(in_pos_files no)
+		(dnp yes)
 		(fields_autoplaced yes)
 		(property "Reference" "J7"
@@
 		(in_bom no)
 		(on_board yes)
-		(in_pos_files yes)
+		(in_pos_files no)
 		(dnp no)
 		(fields_autoplaced yes)
