File: keyboard/keyboard.kicad_pcb (KiCad board)
At the start: 2 copper layers, 98 x 141.5 mm, 83 parts, among them J1 Conn_01x14, J3 OLED, J9 Conn_01x02, SW1 SW_Push, SW10 SW_Push, SW11 SW_Push, SW12 SW_Push, SW13 SW_Push, SW14 SW_Push, SW15 SW_Push, SW16 SW_Push, SW17 SW_Push, SW18 SW_Push, SW19 SW_Push, SW2 SW_Push, SW20 SW_Push, SW21 SW_Push, SW22 SW_Push, SW23 SW_Push, SW24 SW_Push, SW25 SW_Push, SW26 SW_Push, SW27 SW_Push, SW28 SW_Push, SW29 SW_Push, SW3 SW_Push, SW30 SW_Push, SW31 SW_Push, SW32 SW_Push, SW33 SW_Push, SW34 SW_Push, SW4 SW_Push, SW5 SW_Push, SW6 SW_Push, SW7 SW_Push, SW8 SW_Push, SW9 SW_Push

Commit message: keyboard done
Parts:
- removed C15: 100nF, Capacitor_SMD:C_0402_1005Metric
- removed D38: D, Diode_SMD:D_SOD-323
- removed J1: Conn_01x14, Connector_PinHeader_2.54mm:PinHeader_1x14_P2.54mm_Vertical
- removed J3: OLED, Local:2.42-or-2.7-OLED-SSD1309-or-SSD1363
- removed J9: Conn_01x02, Connector_PinHeader_2.54mm:PinHeader_1x02_P2.54mm_Vertical
- removed R24: 100k, Resistor_SMD:R_0402_1005Metric
- added J5: Conn_01x15, Connector_PinHeader_2.54mm:PinHeader_1x15_P2.54mm_Vertical, F.Cu at (107.5, 95.0)
- added J6: Conn_01x15, Connector_FFC-FPC:TE_1-84952-5_1x15-1MP_P1.0mm_Horizontal, B.Cu at (81.5, 98.7)
- moved H3 43.0 mm to (154.0, 94.5)
- moved H4 43.0 mm to (62.0, 94.5)
Connections:
- D30 pad 2: Net-(D30-A) -> WAKEUP
- SW30 pad 2: Net-(D30-A) -> WAKEUP
Routing:
- net WAKEUP: track 0.00 -> 183.7 mm
- net Net-(D30-A): track 177.6 -> 0.00 mm
- net COL1: track 127.5 -> 193.5 mm, vias 0 -> 1
- net COL4: track 161.7 -> 224.4 mm
- net +3V3: track 0.00 -> 60.7 mm, vias 0 -> 1
- net GND: track 0.00 -> 57.5 mm, vias 0 -> 59
- net ROW1: track 135.5 -> 191.6 mm
- net ROW2: track 154.3 -> 209.0 mm
- net ROW3: track 185.9 -> 238.9 mm
- net ROW0: track 97.1 -> 148.6 mm
- net ROW4: track 206.3 -> 255.4 mm
- net COL2: track 131.0 -> 177.8 mm
- net ROW5: track 219.8 -> 266.3 mm
- net ROW6: track 260.9 -> 304.4 mm, vias 2 -> 1
- net COL3: track 147.6 -> 172.7 mm
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- added copper zone on B.Cu, net GND
- added copper zone on F.Cu, net GND
Other:
- board size 98 x 141.5 mm -> 98 x 143.5 mm

Commit message: all checks pass
Parts:
- moved H3 0.50 mm to (154.0, 95.0)
- moved H4 0.50 mm to (62.0, 95.0)
Routing:
- net ROW5: track 266.3 -> 265.7 mm
- net WAKEUP: track 183.7 -> 183.0 mm
- net ROW6: track 304.4 -> 303.7 mm
- net ROW4: track 255.4 -> 254.8 mm
- net COL4: track 224.4 -> 223.8 mm
- net ROW3: track 238.9 -> 238.3 mm
Other:
- board size 98 x 143.5 mm -> 98 x 143 mm
