File: mainboard/mainboard.kicad_pcb (KiCad board)
At the start: 4 copper layers, 98 x 52 mm, 60 parts, among them J1 Conn_01x14, J2 Conn_02x06_Top_Bottom, J3 OLED, J4 TYPE-C-31-M-12, J6 Conn_01x05, J7 SHF-105-01-L-D-RA, J8 Conn_01x02, Q1 AO3400A, SW1 SW_Push, SW35 SW_Push, SW36 SW_Push, U1 RP2350A, U2 W25Q128JVSIQ, U3 MCP73832-2-OT, U8 XC6206P332MR-G, Y1 ABM8-272-T3

Commit message: keyboard done
Parts:
- added H1: MountingHole, MountingHole:MountingHole_2.2mm_M2, F.Cu at (92.0, 108.5)
- added H2: MountingHole, MountingHole:MountingHole_2.2mm_M2, F.Cu at (92.0, 114.4)
- added H5: MountingHole, MountingHole:MountingHole_2.2mm_M2, F.Cu at (97.9, 108.5)
- added H6: MountingHole, MountingHole:MountingHole_2.2mm_M2, F.Cu at (97.9, 114.4)
- added H7: MountingHole, MountingHole:MountingHole_2.2mm_M2, F.Cu at (103.9, 108.5)
- added H8: MountingHole, MountingHole:MountingHole_2.2mm_M2, F.Cu at (103.9, 114.4)

Commit message: erc
Parts:
- removed H5, H6, H7, H8: MountingHole, MountingHole:MountingHole_2.2mm_M2
- removed J1: Conn_01x14, Connector_PinHeader_2.54mm:PinHeader_1x14_P2.54mm_Vertical
- removed SW1: SW_Push, Switch_Keyboard_Cherry_MX:SW_Cherry_MX_PCB_1.00u
- added C15: 100nF, Capacitor_SMD:C_0402_1005Metric, F.Cu at (87.0, 75.5)
- added D38: D, Diode_SMD:D_SOD-323, F.Cu at (86.5, 80.2)
- added J5: Conn_01x15, Connector_PinHeader_2.54mm:PinHeader_1x15_P2.54mm_Vertical, F.Cu at (102.2, 97.0)
- added R24: 100k, Resistor_SMD:R_0402_1005Metric, F.Cu at (85.0, 75.5)
- moved H2 64.4 mm to (154.0, 97.0)
- moved H1 32.1 mm to (62.0, 97.0)
- moved SW35 1.55 mm to (153.4, 90.5)
- moved J7 0.73 mm to (149.5, 59.0)
- moved C11 0.33 mm to (121.2, 80.2)
Connections:
- J7 pad 10: /nRESET -> unconnected-(J7-Pin_10-Pad10)
Routing:
- net (no net): track 47.1 -> 0.00 mm
- net Net-(D38-A): track 0.00 -> 27.7 mm
- net +3V3: track 42.2 -> 21.2 mm, vias 15 -> 33
- net WAKEUP: track 56.8 -> 44.1 mm
- net ROW0: track 27.0 -> 32.7 mm
- net COL0: track 21.7 -> 27.1 mm
- net ROW3: track 18.2 -> 23.7 mm
- net ROW4: track 18.9 -> 24.4 mm
- net COL4: track 18.6 -> 24.0 mm
- net ROW6: track 23.9 -> 29.4 mm
- net ROW5: track 20.5 -> 25.9 mm
- net ROW2: track 17.7 -> 23.1 mm
- net COL3: track 26.4 -> 31.9 mm
- net ROW1: track 17.1 -> 21.3 mm
- net COL1: track 26.6 -> 30.6 mm
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- added copper zone on B.Cu, net +3V3
- added copper zone on In2.Cu, net +3V3
Other:
- board text removed: "GND"

Commit message: all checks pass
Parts:
- removed D38: D, Diode_SMD:D_SOD-323
- removed R24: 100k, Resistor_SMD:R_0402_1005Metric
- added J9: Conn_01x15, Connector_FFC-FPC:TE_1-84952-5_1x15-1MP_P1.0mm_Horizontal, B.Cu at (81.5, 66.8)
- moved C15 13.2 mm to (100.1, 73.9), turned to 90 degrees
- moved J4 8.80 mm to (106.9, 51.5)
- moved R11 8.80 mm to (109.2, 57.5)
- moved R3 8.80 mm to (104.4, 57.5)
- moved J5 5.18 mm to (107.4, 97.0)
- moved R8 1.93 mm to (120.7, 70.5)
- moved R7 1.90 mm to (119.9, 71.2)
Connections:
- J5 pad 1: Net-(D38-A) -> WAKEUP
Routing:
- net COL1: track 30.6 -> 94.6 mm
- net COL2: track 30.4 -> 93.8 mm
- net COL3: track 31.9 -> 93.0 mm
- net ROW0: track 32.7 -> 92.4 mm
- net ROW1: track 21.3 -> 79.1 mm
- net ROW2: track 23.1 -> 78.7 mm
- net ROW3: track 23.7 -> 78.6 mm
- net WAKEUP: track 44.1 -> 98.5 mm, vias 0 -> 2
- net COL4: track 24.0 -> 78.0 mm
- net ROW4: track 24.4 -> 77.3 mm
- net ROW5: track 25.9 -> 76.2 mm
- net COL0: track 27.1 -> 76.7 mm
- net ROW6: track 29.4 -> 77.0 mm
- net Net-(D38-A): track 27.7 -> 0.00 mm
- net VBUS: track 67.8 -> 58.5 mm
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Other:
- outline, holes or cut-outs redrawn
- board text added: "3V3"
- board text added: "BOOT"
- board text added: "GND"
- board text added: "RUN"

Commit message: final changes
Parts:
- R10: value 0 -> 0R; footprint Resistor_SMD:R_0402_1005Metric -> Resistor_SMD:R_0603_1608Metric
- SW35, SW36: footprint Button_Switch_SMD:SW_Push_1P1T_NO_Vertical_Wuerth_434133025816 -> Button_Switch_SMD:SW_Push_1P1T_XKB_TS-1187A
- moved J7 0.99 mm to (149.5, 58.0)
- moved R10 0.38 mm to (103.0, 71.3)
- moved SW36 0.33 mm to (153.5, 70.4)
- moved SW35 0.28 mm to (153.4, 90.8)
Routing:
- net /SWD: track 53.9 -> 48.2 mm
- net /SWCLK: track 49.9 -> 45.7 mm
- net Net-(R4-Pad1): track 9.29 -> 11.8 mm
- net GND: track 68.1 -> 69.6 mm
- net Net-(D35-A): track 91.1 -> 92.2 mm
- net /RUN: track 29.7 -> 30.6 mm
- net /~{USB_BOOT}: track 59.3 -> 60.1 mm
Other:
- board text added: "1"
