File: mainboard/mainboard.kicad_sch (KiCad schematic)
At the start: 46 parts, among them J1 Conn_01x14, J2 Conn_02x06_Top_Bottom, J3 OLED, J6 Conn_01x05, J7 SHF-105-01-L-D-RA, SW35 SW_Push, SW36 SW_Push, U1 RP2350A, U2 W25Q128JVSIQ, Y1 ABM8-272-T3

Commit message: split
Other:
- removed sheet Matrix

Commit message: keyboard done
Parts:
- removed J1: Conn_01x14, Connector_PinHeader_2.54mm:PinHeader_1x14_P2.54mm_Vertical, symbol Connector_Generic:Conn_01x14
- added C15: 100nF, Capacitor_SMD:C_0402_1005Metric, symbol Device:C
- added D38: D, Diode_SMD:D_SOD-323, symbol Device:D_Small
- added J5: Conn_01x15, Connector_PinHeader_2.54mm:PinHeader_1x15_P2.54mm_Vertical, symbol Connector_Generic:Conn_01x15
- added R24: 100k, Resistor_SMD:R_0402_1005Metric, symbol Device:R
Connections:
- net +3V3: now also J5.15 (Pin_15), R24.1
- net COL0: now also J5.3 (Pin_3)
- net COL1: now also J5.13 (Pin_13)
- net COL2: now also J5.12 (Pin_12)
- net COL3: now also J5.11 (Pin_11)
- net COL4: now also J5.6 (Pin_6)
- net GND: now also C15.2, J5.14 (Pin_14)
- net ROW0: now also J5.10 (Pin_10)
- net ROW1: now also J5.9 (Pin_9)
- net ROW2: now also J5.8 (Pin_8)
- net ROW3: now also J5.7 (Pin_7)
- net ROW4: now also J5.5 (Pin_5)
- net ROW5: now also J5.4 (Pin_4)
- net ROW6: now also J5.2 (Pin_2)
- net WAKEUP: now also C15.1, D38.1 (K), R24.2
- new net: D38.2 (A), J5.1 (Pin_1)
Other:
- note removed: "Backup"
- moved on the sheet: J3

Commit message: erc
Parts:
- removed H5, H6, H7, H8: MountingHole, MountingHole:MountingHole_2.2mm_M2, symbol Mechanical:MountingHole
Connections:
- net nRESET: no longer names the net of J7.10 (Pin_10)
- no-connect marks 3 -> 4
Other:
- note added: "nRST"

Commit message: all checks pass
Parts:
- removed D38: D, Diode_SMD:D_SOD-323, symbol Device:D_Small
- removed R24: 100k, Resistor_SMD:R_0402_1005Metric, symbol Device:R
- added J9: Conn_01x15, Connector_FFC-FPC:TE_1-84952-5_1x15-1MP_P1.0mm_Horizontal, symbol Connector_Generic:Conn_01x15
- C15: now not fitted
Connections:
- net +3V3: now also J9.1 (Pin_1)
- net COL0: now also J9.13 (Pin_13)
- net COL1: now also J9.3 (Pin_3)
- net COL2: now also J9.4 (Pin_4)
- net COL3: now also J9.5 (Pin_5)
- net COL4: now also J9.10 (Pin_10)
- net GND: now also J9.2 (Pin_2)
- net ROW0: now also J9.6 (Pin_6)
- net ROW1: now also J9.7 (Pin_7)
- net ROW2: now also J9.8 (Pin_8)
- net ROW3: now also J9.9 (Pin_9)
- net ROW4: now also J9.11 (Pin_11)
- net ROW5: now also J9.12 (Pin_12)
- net ROW6: now also J9.14 (Pin_14)
- net WAKEUP: now also J5.1 (Pin_1), J9.15 (Pin_15)
Other:
- note added: "Neither of buttons are strictly necessary (though the BOOTSEL button would have to be replaced with a header or similar if USB boot mode was required), and can be removed, but they certainly make using the RP2350 a far more pleasant experience."
- note added: "took notes from RP2350A_Minimal_USBC"

Commit message: final changes
Parts:
- BZ1, C15, R1, R9: now left out of the parts list
- J7: now fitted; now left out of the parts list
- R10: value 0 -> 0R; footprint Resistor_SMD:R_0402_1005Metric -> Resistor_SMD:R_0603_1608Metric; LCSC (none) -> C21189
- R2, R4, R6: LCSC (none) -> C11702
- R5, R7, R8: LCSC (none) -> C25105
- SW35, SW36: footprint Button_Switch_SMD:SW_Push_1P1T_NO_Vertical_Wuerth_434133025816 -> Button_Switch_SMD:SW_Push_1P1T_XKB_TS-1187A; LCSC (none) -> C318884
